Commit message: Bringup and model

File: src/rubot_mecanum_description/urdf/rubot0.urdf (robot description, URDF)
Before this commit: robot nexus, 8 links, 7 joints
Links:
- link lower_left_wheel: mass 0.05 -> 0.3844
- link lower_right_wheel: mass 0.05 -> 0.3844
- link upper_right_wheel: mass 0.05 -> 0.3844

Commit message: rubot0

File: src/rubot_mecanum_description/urdf/rubot0.urdf (robot description, URDF)
Before this commit: robot rUBot, 8 links, 7 joints
Joints:
- joint joint_camera: origin xyz=0.130 0.0 0.072 rpy=0 0 0 -> xyz=0 0 0 rpy=0 0 0
- joint lower_left_wheel_joint: origin xyz=-0.082 0.106 -0.028 rpy=0 0 0 -> xyz=0 0 0 rpy=0 0 0
- joint lower_right_wheel_joint: origin xyz=-0.082 -0.106 -0.028 rpy=0 0 0 -> xyz=0 0 0 rpy=0 0 0
- joint scan_joint: origin xyz=0.0 -0.0 0.04 rpy=0 0 0 -> xyz=0.13 0.075 0.16 rpy=0 0 0
- joint upper_left_wheel_joint: origin xyz=0.073 0.106 -0.028 rpy=0 0 0 -> xyz=0 0 0 rpy=0 0 0
- joint upper_right_wheel_joint: origin xyz=0.073 -0.106 -0.028 rpy=0 0 0 -> xyz=0 0 0 rpy=0 0 0

Commit message: rubot madel

File: src/rubot_mecanum_description/urdf/rubot0.urdf (robot description, URDF)
Before this commit: robot rUBot, 8 links, 7 joints
Links:
- link base_link: geometry collision mesh filename=package://rubot_mecanum_description/meshes/rubot/base_link.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 scale=0.001 0.001 0.001; visual mesh filename=package://rubot_mecanum_description/meshes/rubot/base_link.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 scale=0.001 0.001 0.001
- link base_scan: geometry collision cylinder length=0.03 radius=0.05; visual mesh filename=package://rubot_mecanum_description/meshes/rubot/lidar.stl scale=0.001 0.001 0.001
