Commit message: slam i rubot model

File: src/rubot_mecanum_description/urdf/rubot_rp.urdf (robot description, URDF)
Before this commit: robot nexus, 8 links, 7 joints
Links:
- link base_scan: geometry collision cylinder length=0.01575 radius=0.0275; visual mesh filename=package://rubot_mecanum_description/meshes/rubot/Lidar.stl scale=0.001 0.001 0.001
- link camera: mass 1e-3 -> 1; geometry collision box size=0.075 0.075 0.025; visual mesh filename=package://rubot_mecanum_description/meshes/rubot/piCamera.s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 scale=0.001 0.001 0.001
- link lower_left_wheel: geometry collision mesh filename=package://rubot_mecanum_description/meshes/rubot/lower_left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 scale=0.001 0.001 0.001; visual mesh filename=package://rubot_mecanum_description/meshes/rubot/lower_left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 scale=0.001 0.001 0.001
- link lower_right_wheel: geometry collision mesh filename=package://rubot_mecanum_description/meshes/rubot/lower_righ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 scale=0.001 0.001 0.001; visual mesh filename=package://rubot_mecanum_description/meshes/rubot/lower_righ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 scale=0.001 0.001 0.001
- link upper_left_wheel: geometry collision mesh filename=package://rubot_mecanum_description/meshes/rubot/upper_left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 scale=0.001 0.001 0.001; visual mesh filename=package://rubot_mecanum_description/meshes/rubot/upper_left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 scale=0.001 0.001 0.001
- link upper_right_wheel: geometry collision mesh filename=package://rubot_mecanum_description/meshes/rubot/upper_righ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 scale=0.001 0.001 0.001; visual mesh filename=package://rubot_mecanum_description/meshes/rubot/upper_righ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 scale=0.001 0.001 0.001
Joints:
- joint joint_camera: origin xyz=0.236 0.076 0.072 rpy=0 0 0 -> xyz=0.120 0.0 0.09 rpy=0 0 0
- joint lower_left_wheel_joint: origin xyz=0 0 0 rpy=0 0 0 -> xyz=-0.085 0.1 0 rpy=0 0 0
- joint lower_right_wheel_joint: origin xyz=0 0 0 rpy=0 0 0 -> xyz=-0.085 -0.1 0 rpy=0 0 0
- joint scan_joint: origin xyz=0.111 0.076 0.124 rpy=0 0 3.14 -> xyz=0 0 0.15 rpy=0 0 3.14
- joint upper_left_wheel_joint: origin xyz=0 0 0 rpy=0 0 0 -> xyz=0.07 0.1 0 rpy=0 0 0
- joint upper_right_wheel_joint: origin xyz=0 0 0 rpy=0 0 0 -> xyz=0.07 -0.1 0 rpy=0 0 0

Commit message: rubot rp model colision modification

File: src/rubot_mecanum_description/urdf/rubot_rp.urdf (robot description, URDF)
Before this commit: robot nexus, 8 links, 7 joints
Links:
- link base_link: geometry collision box size=0.26 0.15 0.1; visual mesh filename=package://rubot_mecanum_description/meshes/rubot/base_link.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 scale=0.001 0.001 0.001

Commit message: rubot model

File: src/rubot_mecanum_description/urdf/rubot_rp.urdf (robot description, URDF)
Before this commit: robot rubot, 8 links, 7 joints
Links:
- link base_link: geometry collision box size=0.26 0.15 0.09; visual mesh filename=package://rubot_mecanum_description/meshes/rubot/base_link.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 scale=0.001 0.001 0.001
- link lower_left_wheel: geometry collision cylinder length=0.03 radius=0.05; visual mesh filename=package://rubot_mecanum_description/meshes/rubot/lower_left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 scale=0.001 0.001 0.001
- link lower_right_wheel: geometry collision cylinder length=0.03 radius=0.05; visual mesh filename=package://rubot_mecanum_description/meshes/rubot/lower_righ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 scale=0.001 0.001 0.001
- link upper_left_wheel: geometry collision cylinder length=0.03 radius=0.05; visual mesh filename=package://rubot_mecanum_description/meshes/rubot/upper_left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 scale=0.001 0.001 0.001
- link upper_right_wheel: geometry collision cylinder length=0.03 radius=0.05; visual mesh filename=package://rubot_mecanum_description/meshes/rubot/upper_righ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 scale=0.001 0.001 0.001

Commit message: wheels turning

File: src/rubot_mecanum_description/urdf/rubot_rp.urdf (robot description, URDF)
Before this commit: robot rubot, 8 links, 7 joints
Links:
- link base_link: geometry collision box size=0.26 0.15 0.12; visual mesh filename=package://rubot_mecanum_description/meshes/rubot/base_link.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 scale=0.001 0.001 0.001
- link lower_left_wheel: geometry collision cylinder length=0.03 radius=0.06; visual mesh filename=package://rubot_mecanum_description/meshes/rubot/lower_left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 scale=0.001 0.001 0.001
- link lower_right_wheel: geometry collision cylinder length=0.03 radius=0.06; visual mesh filename=package://rubot_mecanum_description/meshes/rubot/lower_righ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 scale=0.001 0.001 0.001
- link upper_left_wheel: geometry collision cylinder length=0.03 radius=0.06; visual mesh filename=package://rubot_mecanum_description/meshes/rubot/upper_left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 scale=0.001 0.001 0.001
- link upper_right_wheel: geometry collision cylinder length=0.03 radius=0.06; visual mesh filename=package://rubot_mecanum_description/meshes/rubot/upper_righ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 scale=0.001 0.001 0.001

Commit message: model rubot mu and pid

File: src/rubot_mecanum_description/urdf/rubot_rp.urdf (robot description, URDF)
Before this commit: robot rubot, 8 links, 7 joints
Links:
- link base_link: mass 2 -> 5; geometry collision box size=0.23 0.12 0.05; visual mesh filename=package://rubot_mecanum_description/meshes/rubot/base_link.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 scale=0.001 0.001 0.001
- link base_scan: mass 0.057 -> 0.05; geometry collision cylinder length=0.05 radius=0.05; visual mesh filename=package://rubot_mecanum_description/meshes/rubot/Lidar.stl scale=0.001 0.001 0.001
- link camera: mass 1 -> 0.01
- link lower_left_wheel: mass 0.05 -> 0.1; geometry collision cylinder length=0.03 radius=0.05; visual mesh filename=package://rubot_mecanum_description/meshes/rubot/lower_left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 scale=0.001 0.001 0.001
- link lower_right_wheel: mass 0.05 -> 0.1; geometry collision cylinder length=0.03 radius=0.05; visual mesh filename=package://rubot_mecanum_description/meshes/rubot/lower_righ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 scale=0.001 0.001 0.001
- link upper_left_wheel: mass 0.05 -> 0.1; geometry collision cylinder length=0.03 radius=0.05; visual mesh filename=package://rubot_mecanum_description/meshes/rubot/upper_left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 scale=0.001 0.001 0.001
- link upper_right_wheel: mass 0.05 -> 0.1; geometry collision cylinder length=0.03 radius=0.05; visual mesh filename=package://rubot_mecanum_description/meshes/rubot/upper_righ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 scale=0.001 0.001 0.001

Commit message: urdf collisions

File: src/rubot_mecanum_description/urdf/rubot_rp.urdf (robot description, URDF)
Before this commit: robot rubot, 8 links, 7 joints
Links:
- link camera: geometry collision box size=0.05 0.05 0.025; visual mesh filename=package://rubot_mecanum_description/meshes/rubot/piCamera.s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 scale=0.001 0.001 0.001
- link lower_left_wheel: geometry collision cylinder length=0.03 radius=0.055; visual mesh filename=package://rubot_mecanum_description/meshes/rubot/lower_left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 scale=0.001 0.001 0.001
- link lower_right_wheel: geometry collision cylinder length=0.03 radius=0.055; visual mesh filename=package://rubot_mecanum_description/meshes/rubot/lower_righ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 scale=0.001 0.001 0.001
- link upper_left_wheel: geometry collision cylinder length=0.03 radius=0.055; visual mesh filename=package://rubot_mecanum_description/meshes/rubot/upper_left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 scale=0.001 0.001 0.001
- link upper_right_wheel: geometry collision cylinder length=0.03 radius=0.055; visual mesh filename=package://rubot_mecanum_description/meshes/rubot/upper_righ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 scale=0.001 0.001 0.001

Commit message: inertia rubot

File: src/rubot_mecanum_description/urdf/rubot_rp.urdf (robot description, URDF)
Before this commit: robot rubot, 8 links, 7 joints
Links:
- link lower_left_wheel: mass 0.1 -> 0.2
- link lower_right_wheel: mass 0.1 -> 0.2
- link upper_left_wheel: mass 0.1 -> 0.2
- link upper_right_wheel: mass 0.1 -> 0.2
Joints:
- joint lower_right_wheel_joint: axis 0 1 0 -> 0 -1 0; origin xyz=-0.085 -0.1 0 rpy=0 0 0 -> xyz=-0.085 -0.1 0 rpy=0 0 3.14
- joint upper_right_wheel_joint: axis 0 1 0 -> 0 -1 0; origin xyz=0.07 -0.1 0 rpy=0 0 0 -> xyz=0.07 -0.1 0 rpy=0 0 3.14

Commit message: time correction

File: src/rubot_mecanum_description/urdf/rubot_rp.urdf (robot description, URDF)
Before this commit: robot rubot, 8 links, 7 joints
Links:
- added link part, mass 0.01; collision box size=0.05 0.05 0.025; visual box size=0.05 0.05 0.025
Joints:
- added joint joint_part: type fixed, parent base_link, child part, origin xyz=-0.10 0.0 0.09 rpy=0 0 0
