Commit message: model

File: src/rubot_mecanum_description/urdf/rubot.urdf (robot description, URDF)
Before this commit: robot nexus, 8 links, 7 joints
Links:
- link base_scan: geometry collision cylinder length=0.01575 radius=0.0275; visual mesh filename=package://rubot_mecanum_description/meshes/rubot/lidar.stl scale=0.0015 0.0015 0.0015
Joints:
- joint joint_camera: origin xyz=0.236 0.076 0.072 rpy=0 0 0 -> xyz=0.130 0.0 0.072 rpy=0 0 0
- joint lower_left_wheel_joint: origin xyz=0 0 0 rpy=0 0 0 -> xyz=-0.082 0.106 -0.028 rpy=0 0 0
- joint lower_right_wheel_joint: origin xyz=0 0 0 rpy=0 0 0 -> xyz=-0.082 -0.106 -0.028 rpy=0 0 0
- joint scan_joint: origin xyz=0.111 0.076 0.124 rpy=0 0 0 -> xyz=0.0 -0.0 0.04 rpy=0 0 0
- joint upper_left_wheel_joint: origin xyz=0 0 0 rpy=0 0 0 -> xyz=0.073 0.106 -0.028 rpy=0 0 0
- joint upper_right_wheel_joint: origin xyz=0 0 0 rpy=0 0 0 -> xyz=0.073 -0.106 -0.028 rpy=0 0 0

Commit message: model and ino

File: src/rubot_mecanum_description/urdf/rubot.urdf (robot description, URDF)
Before this commit: robot rubot, 9 links, 8 joints
Joints:
- joint scan_joint: origin xyz=0 0 0.15 rpy=0 0 3.14 -> xyz=0 0 0.15 rpy=0 0 0
