Commit message: models and rubot

File: Documentation/files/Doc/Robot_Models/rubot.urdf (robot description, URDF)
Before this commit: robot rubot, 9 links, 8 joints
Links:
- link part: geometry collision box size=0.05 0.05 0.025; visual box size=0.05 0.05 0.025
Joints:
- joint scan_joint: origin xyz=0 0 0.15 rpy=0 0 3.14 -> xyz=0 0 0.15 rpy=0 0 0

File: src/rubot_mecanum_description/urdf/rubot.urdf (robot description, URDF)
Before this commit: robot rubot, 9 links, 8 joints
Links:
- link camera: geometry collision box size=0.05 0.05 0.025; visual mesh filename=package://rubot_mecanum_description/meshes/rubot/Camera.stl scale=0.001 0.001 0.001
- link part: geometry collision box size=0.05 0.05 0.025; visual mesh filename=package://rubot_mecanum_description/meshes/rubot/number2.stl scale=0.0008 0.0008 0.0008
Joints:
- joint scan_joint: origin xyz=0 0 0.15 rpy=0 0 0 -> xyz=0 0 0.15 rpy=0 0 3.14
