Commit message: limo

File: src/rubot_mecanum_description/urdf/limo/limo_four_diff.xacro (robot description, xacro)
@@ -1,6 +1,6 @@
 <?xml version="1.0"?>
 <robot name="limo_four_diff" xmlns:xacro="http://ros.org/wiki/xacro">
-    <xacro:include filename="$(find limo_description)/urdf/limo_xacro.xacro" />
-    <xacro:include filename="$(find limo_description)/urdf/limo_four_diff.gazebo" />
+    <xacro:include filename="$(find rubot_mecanum_description)/urdf/limo/limo_xacro.xacro" />
+    <xacro:include filename="$(find rubot_mecanum_description)/urdf/limo/limo_four_diff.gazebo" />
     <!-- Variables -->
     <xacro:property name="M_PI" value="3.14159"/>
@@ -22,5 +22,5 @@
             <origin xyz="0 0 -0.15" rpy="0 0 1.57" />
             <geometry>
-                <mesh filename="package://limo_description/meshes/limo_base.dae"/>
+                <mesh filename="package://rubot_mecanum_description/meshes/limo/limo_base.dae"/>
             </geometry>
         </visual>
@@ -28,5 +28,5 @@
             <origin xyz="0 0 -0.15" rpy="0 0 1.57" />
             <geometry>
-                <mesh filename="package://limo_description/meshes/limo_collision.stl"/>
+                <mesh filename="package://rubot_mecanum_description/meshes/limo/limo_collision.stl"/>
             </geometry>
         </collision>

File: src/rubot_mecanum_description/urdf/limo/limo_xacro.xacro (robot description, xacro)
@@ -11,5 +11,5 @@
                 <origin xyz="0 0 0" rpy="0 0 0" />
                 <geometry>
-                    <mesh filename="package://limo_description/meshes/limo_wheel.dae" />
+                    <mesh filename="package://rubot_mecanum_description/meshes/limo/limo_wheel.dae" />
                 </geometry>
             </visual>
